File: Hardware/InkTime_2D-PCB.brd (EAGLE design)
At the start: 46 x 35 mm, 105 parts, among them IC1 BQ25180YBGR, IC2 DRV2605YZFR, IC3 BMA421, IC9 RT6160AWSC, J1 503480-2400, J2 TC2030-IDC, J4 KH-TYPE-C-16P, Q1 20V/4.2A/52mΩ/1.4W, Q3 ESP32_C6_LIBRARY_6_SI1308EDL-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, U1 NRF52840_QF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

Commit message: Updated 2D-PCB Fixes #6
Parts:
- moved ANT1 1.03 mm to (89.5, 143.5)
- moved C15 0.20 mm to (92.5, 140.4)
Routing:
- net GND: track 371.2 -> 350.7 mm, vias 14 -> 29
- net P1.02/1.6C: track 17.6 -> 11.3 mm, vias 2 -> 0
- net P0.14/1.5D: track 20.2 -> 14.5 mm, vias 2 -> 0
- net LX1: track 29.1 -> 32.8 mm
- net 3V3/2.4A: track 125.8 -> 128.8 mm
- net RESE: track 20.3 -> 17.5 mm
- net P0.13/1.5D: track 25.9 -> 28.1 mm
- net RF: track 8.39 -> 9.78 mm
- net SWDCLK: track 46.9 -> 46.3 mm
- net PREVGH: track 21.7 -> 22.2 mm, vias 4 -> 3
- added copper zone on layer 16, net GND
- added copper zone on layer 2, net GND
Other:
- outline, holes or cut-outs redrawn
