File: Hardware/InkTime Schematic.sch (EAGLE design)
At the start: 105 parts, among them IC1 BQ25180YBGR, IC2 DRV2605YZFR, IC3 BMA421, IC9 RT6160AWSC, J1 503480-2400, J2 TC2030-IDC, J4 KH-TYPE-C-16P, Q1 20V/4.2A/52mΩ/1.4W, Q3 ESP32_C6_LIBRARY_6_SI1308EDL-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, U1 NRF52840_QF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

Commit message: Update Schematic
Fixes #5
Parts:
- D2, D5: value ESP32_C6_LIBRARY_5_MBR0530 -> MBR0530
- Q3: value ESP32_C6_LIBRARY_6_SI1308EDL-T1-GE3 -> SI1308EDL-T1-GE3
